Commit message: made urdf independent of lunabot_one

File: description/oak_d_s2.xacro (robot description, xacro)
@@ -38,7 +38,4 @@
         </inertial>
     </link>
-    <gazebo reference="oak_link">
-        <material>Gazebo/DarkGrey</material>
-    </gazebo>
     <!-- RGB camera optical frame (X=right, Y=down, Z=forward) -->
     <joint name="oak_d_rgb_optical_joint" type="fixed">

File: description/robot.urdf.xacro (robot description, xacro)
@@ -1,6 +1,6 @@
 <?xml version="1.0"?>
 <robot xmlns:xacro="http://www.ros.org/wiki/xacro" name="lunabot">
-    <!-- Include robot chassis and wheels from lunabot_one -->
-    <xacro:include filename="$(find lunabot_one)/description/robot_core.xacro"/>
+    <!-- Include robot chassis and wheels -->
+    <xacro:include filename="robot_core.xacro"/>
     <!-- Include OAK-D S2 camera (mounts to chassis) -->
     <xacro:include filename="oak_d_s2.xacro"/>

Commit message: More nav2 implementation, URDF and Launch file implementations

File: description/oak_d_s2.xacro (robot description, xacro)
@@ -13,9 +13,13 @@
     <joint name="oak_d_camera_joint" type="fixed">
         <parent link="chassis"/>
-        <child link="oak_link"/>
+        <child link="oak"/>
         <!-- Front of chassis (x=chassis_length), centered (y=0), on top (z=chassis_height + half camera height) -->
         <origin xyz="${chassis_length} 0 ${chassis_height + oak_d_height/2}" rpy="0 0 0"/>
     </joint>
-    <link name="oak_link">
+    <!-- Frame name "oak" matches depthai_ros_driver node name.
+         The depthai driver publishes calibrated optical frames (oak_rgb_camera_optical_frame,
+         oak_right_camera_optical_frame, oak_imu_frame, etc.) from this root frame.
+         Do NOT define optical frames here — let depthai handle them from calibration data. -->
+    <link name="oak">
         <visual>
             <geometry>
@@ -38,24 +42,3 @@
         </inertial>
     </link>
-    <!-- RGB camera optical frame (X=right, Y=down, Z=forward) -->
-    <joint name="oak_d_rgb_optical_joint" type="fixed">
-        <parent link="oak_link"/>
-        <child link="oak_d_rgb_camera_optical_frame"/>
-        <origin xyz="0 0 0" rpy="${-pi/2} 0 ${-pi/2}"/>
-    </joint>
-    <link name="oak_d_rgb_camera_optical_frame"/>
-    <!-- Stereo/depth optical frame (same as RGB for the S2) -->
-    <joint name="oak_d_stereo_optical_joint" type="fixed">
-        <parent link="oak_link"/>
-        <child link="oak_stereo_camera_optical_frame"/>
-        <origin xyz="0 0 0" rpy="${-pi/2} 0 ${-pi/2}"/>
-    </joint>
-    <link name="oak_stereo_camera_optical_frame"/>
-    <!-- IMU frame (colocated with oak_link) -->
-    <joint name="oak_d_imu_joint" type="fixed">
-        <parent link="oak_link"/>
-        <child link="oak_imu_frame"/>
-        <origin xyz="0 0 0" rpy="0 0 0"/>
-    </joint>
-    <link name="oak_imu_frame"/>
 </robot>

Commit message: Fix OAK-D optical frame TF (split URDF/driver at oak_mount)

File: description/oak_d_s2.xacro (robot description, xacro)
@@ -13,13 +13,12 @@
     <joint name="oak_d_camera_joint" type="fixed">
         <parent link="chassis"/>
-        <child link="oak"/>
+        <child link="oak_mount"/>
         <!-- Front of chassis (x=chassis_length), centered (y=0), on top (z=chassis_height + half camera height) -->
         <origin xyz="${chassis_length} 0 ${chassis_height + oak_d_height/2}" rpy="0 0 0"/>
     </joint>
-    <!-- Frame name "oak" matches depthai_ros_driver node name.
-         The depthai driver publishes calibrated optical frames (oak_rgb_camera_optical_frame,
-         oak_right_camera_optical_frame, oak_imu_frame, etc.) from this root frame.
-         Do NOT define optical frames here — let depthai handle them from calibration data. -->
-    <link name="oak">
+    <!-- URDF owns "oak_mount" (the physical mount point with visual/inertia).
+         depthai_ros_driver publishes oak_mount -> oak -> oak_rgb_camera_optical_frame etc.
+         from calibration data (see camera.i_tf_parent_frame in oak_d_camera.yaml). -->
+    <link name="oak_mount">
         <visual>
             <geometry>
