Commit message: feat(description): size the robot to the 2027 design
Chassis and wheel placeholders replaced with the team's 2027 design
model (ryan-hay.com/rover-sim), taken as a guideline rather than a
measurement and marked "design" in properties.xacro until the built
rover can be measured:

  wheel radius 0.10 -> 0.15 m, width 0.08 -> 0.09 m, mass 1.5 -> 0.85 kg
  track        0.50 -> 0.554 m, wheelbase 0.44 -> 0.62 m
  chassis      0.70 x 0.40 -> 0.813 x 0.432 m (32 x 17 in frame)
  chassis mass 25 -> 28.9 kg (32.3 kg dry, less the wheels)

controllers.yaml and isaac_double.py carry the same wheel radius and
track; a new test keeps the double in step with the controller.

The Nav2 footprint covered the chassis only, but the wheels stand
proud of its sides (outer face 0.322 m against a 0.216 m half-width,
and the old placeholders had the same gap). It now covers whichever
reaches further, and the footprint test checks that rule.

Not changed: gear ratio and max wheel speed (the design gives no drive
ratio), CAN IDs, the camera (the design has a rear RealSense D455-class
where this stack has a front OAK-D), and the excavation mechanism.

Verified in Isaac: spawns at 0.155 m, check_stack --drive 18/18, /odom
within 2 mm of ground truth over 0.5 m.

Co-Authored-By: Claude Opus 5.5 <noreply@anthropic.com>

File: src/lunabot_description/urdf/common/properties.xacro (robot description, xacro)
@@ -18,14 +18,30 @@
     ===================================================================
   -->
+  <!--
+    2027 DESIGN VALUES. Chassis and wheel numbers below marked "design" come
+    from the team's 2027 design model (ryan-hay.com/rover-sim, read
+    2026-10-21). That model is a guideline, not a measurement: it is ahead of
+    the build and will drift from it. Replace each with the measured value
+    once the rover exists, and keep controllers.yaml in step.
+  -->
   <!-- ==================== Chassis ==================== -->
   <!-- Body box. base_link sits at its geometric centre, at axle height. -->
-  <xacro:property name="chassis_length" value="0.70"/>   <!-- X, fore-aft -->
-  <xacro:property name="chassis_width"  value="0.40"/>   <!-- Y, lateral  -->
+  <!-- design: 32 x 17 in frame of 2 x 1 in 6061 tube, centred over the axles -->
+  <xacro:property name="chassis_length" value="0.813"/>  <!-- X, fore-aft -->
+  <xacro:property name="chassis_width"  value="0.432"/>  <!-- Y, lateral  -->
+  <!-- PLACEHOLDER. The real frame sits above the axles (21-26 cm off the
+       ground) with the drive units and e-box hanging off it; one box at axle
+       height is a stand-in until the description models those parts. -->
   <xacro:property name="chassis_height" value="0.20"/>   <!-- Z           -->
-  <xacro:property name="chassis_mass"   value="25.0"/>   <!-- kg, everything but wheels -->
+  <!-- design: 32.3 kg dry, less four 0.85 kg wheels. Includes the drum,
+       hopper and actuators, which the description does not model yet. -->
+  <xacro:property name="chassis_mass"   value="28.9"/>   <!-- kg, everything but wheels -->
   <!-- ==================== Wheels ==================== -->
-  <xacro:property name="wheel_radius"    value="0.10"/>
-  <xacro:property name="wheel_width"     value="0.08"/>
-  <xacro:property name="wheel_mass"      value="1.5"/>
+  <!-- design: 0.136 m tread band with 1.4 cm grousers, 9 cm wide. The
+       rolling radius on regolith lies between the band and the grouser tips;
+       0.15 is the tips. Measure it: odometry scales with it directly. -->
+  <xacro:property name="wheel_radius"    value="0.15"/>
+  <xacro:property name="wheel_width"     value="0.09"/>
+  <xacro:property name="wheel_mass"      value="0.85"/>
   <!--
     Lateral distance between the left and right wheel centreplanes.
@@ -35,9 +51,11 @@
     wider than its geometric one. Do not pre-bake the fudge factor here.
   -->
-  <xacro:property name="wheel_separation" value="0.50"/>
+  <!-- design: wheel centreplanes at +-0.277 m -->
+  <xacro:property name="wheel_separation" value="0.554"/>
   <!-- Fore-aft distance between the front and rear axles. Does not enter
        the differential kinematics; it sets where the wheels are drawn and
        how the robot behaves in sim contact. -->
-  <xacro:property name="wheel_base" value="0.44"/>
+  <!-- design: axles 0.62 m apart -->
+  <xacro:property name="wheel_base" value="0.62"/>
   <!-- ==================== OAK-D S2 ==================== -->
   <!-- Enclosure, from the Luxonis datasheet. VERIFY against your unit. -->
@@ -72,5 +90,7 @@
         motor_free_speed_rpm / gear_ratio * 2*pi / 60
     and then measure, because free speed under load is not free speed.
-    16.0 rad/s at r=0.10 m is about 1.6 m/s, which is plausible and unverified.
+    16.0 rad/s at r=0.15 m is about 2.4 m/s, far above the 2027 design's
+    0.3 m/s top speed, so expect this to come down a long way once the drive
+    gearbox ratio is chosen (the design names a 3-stage planetary, no ratio).
   -->
   <xacro:property name="max_wheel_rad_s" value="16.0"/>

Commit message: feat(description): six wheels, drop-centre, so the rover can turn on the spot
The 2026 four-wheeler could not pivot in sand and the 2027 four-wheel
design has the same proportions. Widening the track enough (~0.9 m)
breaks the 0.75 m starting width, so the rover gets a middle axle at the
same 0.62 m wheelbase, wheel_drop (1.5 cm, assumed) lower than the ends.
Its wheels sit on the pivot axis and carry weight without scrubbing.

- properties.xacro: wheel_drop; wheel.xacro takes a z offset.
- ros2_control: middle_left/right_wheel_joint, CAN IDs 5/6 PLACEHOLDERS
  (not wired; assign before hw:=real), right side inverted.
- diff_drive: three wheels a side; wheel_separation_multiplier 1.5 ->
  1.2 (Isaac with sinkage: 85% of a commanded pivot, 74-85% of arcs at
  1.0; 1.5 overshot to 148% on rigid ground).
- Tests and the Isaac double follow the six joint names.

Co-Authored-By: Claude Opus 5.5 <noreply@anthropic.com>

File: src/lunabot_description/urdf/common/properties.xacro (robot description, xacro)
@@ -58,4 +58,18 @@
   <!-- design: axles 0.62 m apart -->
   <xacro:property name="wheel_base" value="0.62"/>
+  <!--
+    SIX wheels, drop-centre: a middle axle at x = 0, wheel_drop LOWER than
+    the front and rear ones. Chosen 2026-10-22 so the rover can turn on the
+    spot in sand, which the 2026 four-wheeler could not do (and the 2027
+    four-wheel design would not either: lunabot_sim/robot/soil.py). The
+    middle wheels sit on the pivot axis, so they carry weight without
+    scrubbing; lowered, they carry more of it, and the ends scrub less.
+    The rover rocks onto the middle axle and one end; by design.
+    NOT in the team's design model yet: the drop is an ASSUMPTION. Too
+    little and the middle carries no extra load; too much and the rover
+    rocks visibly and pitches its camera. 1.5 cm is a starting point for
+    sand, where the middle wheels also sink further.
+  -->
+  <xacro:property name="wheel_drop" value="0.015"/>
   <!-- ==================== OAK-D S2 ==================== -->
   <!-- Enclosure, from the Luxonis datasheet. VERIFY against your unit. -->

File: src/lunabot_description/urdf/lunabot.urdf.xacro (robot description, xacro)
@@ -55,4 +55,9 @@
   <xacro:lunabot_wheel prefix="${prefix}" name="front_right" side="right"
                        x_offset="${wheel_base / 2.0}"/>
+  <!-- Middle axle, dropped: see wheel_drop in properties.xacro. -->
+  <xacro:lunabot_wheel prefix="${prefix}" name="middle_left"  side="left"
+                       x_offset="0" z_offset="${-wheel_drop}"/>
+  <xacro:lunabot_wheel prefix="${prefix}" name="middle_right" side="right"
+                       x_offset="0" z_offset="${-wheel_drop}"/>
   <xacro:lunabot_wheel prefix="${prefix}" name="rear_left"   side="left"
                        x_offset="${-wheel_base / 2.0}"/>

File: src/lunabot_description/urdf/ros2_control/lunabot.ros2_control.xacro (robot description, xacro)
@@ -162,4 +162,11 @@
       <xacro:lunabot_wheel_joint name="front_left_wheel_joint"  can_id="2" invert="false"/>
       <xacro:lunabot_wheel_joint name="front_right_wheel_joint" can_id="1" invert="true"/>
+      <!--
+        Middle axle (six-wheel drop-centre, 2026-10-22). CAN IDs 5 and 6 are
+        PLACEHOLDERS: nothing is wired yet. Assign them with the electrical
+        team before hw:=real.
+      -->
+      <xacro:lunabot_wheel_joint name="middle_left_wheel_joint"  can_id="5" invert="false"/>
+      <xacro:lunabot_wheel_joint name="middle_right_wheel_joint" can_id="6" invert="true"/>
       <xacro:lunabot_wheel_joint name="rear_left_wheel_joint"   can_id="3" invert="false"/>
       <xacro:lunabot_wheel_joint name="rear_right_wheel_joint"  can_id="4" invert="true"/>

File: src/lunabot_description/urdf/wheel.xacro (robot description, xacro)
@@ -9,9 +9,9 @@
     was hardcoded in C++ (right_front_->SetInverted(true)), which meant
     rewiring the robot required recompiling it.
-    All four wheels rotate about their local Y axis. The cylinder is
+    Every wheel rotates about its local Y axis. The cylinder is
     modelled along Z and rotated into place, which is why the inertia
     macro takes an origin block.
   -->
-  <xacro:macro name="lunabot_wheel" params="prefix name side x_offset">
+  <xacro:macro name="lunabot_wheel" params="prefix name side x_offset z_offset:=0">
     <xacro:property name="y_sign" value="${1 if side == 'left' else -1}"/>
     <xacro:property name="y_offset" value="${y_sign * wheel_separation / 2.0}"/>
@@ -51,5 +51,5 @@
       <parent link="${prefix}base_link"/>
       <child  link="${prefix}${name}_wheel_link"/>
-      <origin xyz="${x_offset} ${y_offset} 0" rpy="0 0 0"/>
+      <origin xyz="${x_offset} ${y_offset} ${z_offset}" rpy="0 0 0"/>
       <axis xyz="0 1 0"/>
       <dynamics damping="0.05" friction="0.1"/>
